File: hardware/controller/MEMORY.kicad_sch (KiCad schematic)
At the start: 8 parts, among them IC103 4677, IC104 W25Q256JVEIQ

Commit message: done but need to add stitching vias
Parts:
- TP801: renamed from TP126; footprint TestPoint:TestPoint_Pad_1.0x1.0mm -> 5000; Arrow Part Number (none) -> 5001; Arrow Price/Stock (none) -> https://www.arrow.com/en/products/5001/keystone-electronics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; Manufacturer_Name (none) -> Keystone Electronics; Manufacturer_Part_Number (none) -> 5001; Mouser Part Number (none) -> 534-5001; Mouser Price/Stock (none) -> https://www.mouser.co.uk/ProductDetail/Keystone-Electronics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
- TP802: renamed from TP127; footprint TestPoint:TestPoint_Pad_1.0x1.0mm -> 5000; Arrow Part Number (none) -> 5001; Arrow Price/Stock (none) -> https://www.arrow.com/en/products/5001/keystone-electronics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; Manufacturer_Name (none) -> Keystone Electronics; Manufacturer_Part_Number (none) -> 5001; Mouser Part Number (none) -> 534-5001; Mouser Price/Stock (none) -> https://www.mouser.co.uk/ProductDetail/Keystone-Electronics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
- renumbered C119 to C801, C120 to C802, C121 to C803, C122 to C804, IC103 to IC801, IC104 to IC802
Changed lines of the file:
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@@
 		(dnp no)
 		(fields_autoplaced yes)
-		(property "Reference" "#PWR0163"
+		(property "Reference" "#PWR0801"
 			(at 119.38 96.52 0)
 			(effects
@@
 			(project "controller"
 				(path "/869bea87-c885-4ead-826b-3f34ceacafad/0e7b3f4d-646f-4949-ba8d-4e4489aa7d1d"
-					(reference "#PWR0163")
+					(reference "#PWR0801")
 					(unit 1)
 				)
@@
 		(dnp no)
 		(fields_autoplaced yes)
-		(property "Reference" "C120"
+		(property "Reference" "C802"
 			(at 168.91 115.5699 0)
 			(effects
@@
 			(project "controller"
 				(path "/869bea87-c885-4ead-826b-3f34ceacafad/0e7b3f4d-646f-4949-ba8d-4e4489aa7d1d"
-					(reference "C120")
+					(reference "C802")
 					(unit 1)
 				)
@@
 		(dnp no)
 		(fields_autoplaced yes)
-		(property "Reference" "IC104"
+		(property "Reference" "IC802"
 			(at 139.7 118.11 0)
 			(effects
@@
 			(project "controller"
 				(path "/869bea87-c885-4ead-826b-3f34ceacafad/0e7b3f4d-646f-4949-ba8d-4e4489aa7d1d"
-					(reference "IC104")
+					(reference "IC802")
 					(unit 1)
 				)
@@
 		(on_board yes)
 		(dnp no)
-		(property "Reference" "#PWR0168"
+		(property "Reference" "#PWR0806"
 			(at 176.53 78.74 0)
 			(effects
@@
 			(project "controller"
 				(path "/869bea87-c885-4ead-826b-3f34ceacafad/0e7b3f4d-646f-4949-ba8d-4e4489aa7d1d"
-					(reference "#PWR0168")
+					(reference "#PWR0806")
 					(unit 1)
 				)
@@
 		(dnp no)
 		(fields_autoplaced yes)
-		(property "Reference" "C121"
+		(property "Reference" "C803"
 			(at 180.34 67.3099 0)
 			(effects
@@
 			(project "controller"
 				(path "/869bea87-c885-4ead-826b-3f34ceacafad/0e7b3f4d-646f-4949-ba8d-4e4489aa7d1d"
-					(reference "C121")
+					(reference "C803")
 					(unit 1)
 				)
@@
 		(dnp no)
 		(fields_autoplaced yes)
-		(property "Reference" "IC103"
+		(property "Reference" "IC801"
 			(at 139.7 74.93 0)
 			(effects
@@
 			(project "controller"
 				(path "/869bea87-c885-4ead-826b-3f34ceacafad/0e7b3f4d-646f-4949-ba8d-4e4489aa7d1d"
-					(reference "IC103")
+					(reference "IC801")
 					(unit 1)
 				)
@@
 		(on_board yes)
 		(dnp no)
-		(property "Reference" "#PWR0166"
+		(property "Reference" "#PWR0804"
 			(at 165.1 78.74 0)
 			(effects
@@
 			(project "controller"
 				(path "/869bea87-c885-4ead-826b-3f34ceacafad/0e7b3f4d-646f-4949-ba8d-4e4489aa7d1d"
-					(reference "#PWR0166")
+					(reference "#PWR0804")
 					(unit 1)
 				)
@@
 		(dnp no)
 		(fields_autoplaced yes)
-		(property "Reference" "#PWR0165"
+		(property "Reference" "#PWR0803"
 			(at 139.7 152.4 0)
 			(effects
@@
 			(project "controller"
 				(path "/869bea87-c885-4ead-826b-3f34ceacafad/0e7b3f4d-646f-4949-ba8d-4e4489aa7d1d"
-					(reference "#PWR0165")
+					(reference "#PWR0803")
 					(unit 1)
 				)
@@
 		(on_board yes)
 		(dnp no)
-		(property "Reference" "#PWR0169"
+		(property "Reference" "#PWR0807"
 			(at 176.53 127 0)
 			(effects
@@
 			(project "controller"
 				(path "/869bea87-c885-4ead-826b-3f34ceacafad/0e7b3f4d-646f-4949-ba8d-4e4489aa7d1d"
-					(reference "#PWR0169")
+					(reference "#PWR0807")
 					(unit 1)
 				)
@@
 		(on_board yes)
 		(dnp no)
-		(property "Reference" "#PWR0167"
+		(property "Reference" "#PWR0805"
 			(at 165.1 127 0)
 			(effects
@@
 			(project "controller"
 				(path "/869bea87-c885-4ead-826b-3f34ceacafad/0e7b3f4d-646f-4949-ba8d-4e4489aa7d1d"
-					(reference "#PWR0167")
+					(reference "#PWR0805")
 					(unit 1)
 				)
@@
 		(on_board yes)
 		(dnp no)
-		(property "Reference" "TP127"
+		(property "Reference" "TP802"
 			(at 117.094 118.11 0)
 			(effects
@@
 			)
 		)
-		(property "Footprint" "TestPoint:TestPoint_Pad_1.0x1.0mm"
-			(at 123.19 125.73 0)
-			(effects
-				(font
-					(size 1.27 1.27)
-				)
-				(hide yes)
-			)
-		)
-		(property "Datasheet" "~"
-			(at 123.19 125.73 0)
-			(effects
-				(font
-					(size 1.27 1.27)
-				)
-				(hide yes)
-			)
-		)
-		(property "Description" "test point"
+		(property "Footprint" "5000"
+			(at 134.62 220.65 0)
+			(effects
+				(font
+					(size 1.27 1.27)
+				)
+				(justify left top)
+				(hide yes)
+			)
+		)
+		(property "Datasheet" "http://www.keyelco.com/product-pdf.cfm?p=1310"
+			(at 134.62 320.65 0)
+			(effects
+				(font
+					(size 1.27 1.27)
+				)
+				(justify left top)
+				(hide yes)
+			)
+		)
+		(property "Description" "KEYSTONE - 5001 - TEST POINT, CONNECTOR, BLACK"
 			(at 118.11 125.73 0)
 			(effects
@@
 					(size 1.27 1.27)
 				)
+				(hide yes)
+			)
+		)
+		(property "Height" ""
+			(at 134.62 520.65 0)
+			(effects
+				(font
+					(size 1.27 1.27)
+				)
+				(justify left top)
+				(hide yes)
+			)
+		)
+		(property "Manufacturer_Name" "Keystone Electronics"
+			(at 134.62 620.65 0)
+			(effects
+				(font
+					(size 1.27 1.27)
+				)
+				(justify left top)
+				(hide yes)
+			)
+		)
+		(property "Manufacturer_Part_Number" "5001"
+			(at 134.62 720.65 0)
+			(effects
+				(font
+					(size 1.27 1.27)
+				)
+				(justify left top)
+				(hide yes)
+			)
+		)
+		(property "Mouser Part Number" "534-5001"
+			(at 134.62 820.65 0)
+			(effects
+				(font
+					(size 1.27 1.27)
+				)
+				(justify left top)
+				(hide yes)
+			)
+		)
+		(property "Mouser Price/Stock" "https://www.mouser.co.uk/ProductDetail/Keystone-Electronics/5001?qs=q0tsjPZWdm%2FW0vdr%2FwowKg%3D%3D"
+			(at 134.62 920.65 0)
+			(effects
+				(font
+					(size 1.27 1.27)
+				)
+				(justify left top)
+				(hide yes)
+			)
+		)
+		(property "Arrow Part Number" "5001"
+			(at 134.62 1020.65 0)
+			(effects
+				(font
+					(size 1.27 1.27)
+				)
+				(justify left top)
+				(hide yes)
+			)
+		)
+		(property "Arrow Price/Stock" "https://www.arrow.com/en/products/5001/keystone-electronics?utm_currency=USD&region=europe"
+			(at 134.62 1120.65 0)
+			(effects
+				(font
+					(size 1.27 1.27)
+				)
+				(justify left top)
 				(hide yes)
 			)
@@
 			(project "controller"
 				(path "/869bea87-c885-4ead-826b-3f34ceacafad/0e7b3f4d-646f-4949-ba8d-4e4489aa7d1d"
-					(reference "TP127")
+					(reference "TP802")
 					(unit 1)
 				)
@@
 		(dnp no)
 		(fields_autoplaced yes)
-		(property "Reference" "#PWR0164"
+		(property "Reference" "#PWR0802"
 			(at 119.38 139.7 0)
 			(effects
@@
 			(project "controller"
 				(path "/869bea87-c885-4ead-826b-3f34ceacafad/0e7b3f4d-646f-4949-ba8d-4e4489aa7d1d"
-					(reference "#PWR0164")
+					(reference "#PWR0802")
 					(unit 1)
 				)
@@
 		(dnp no)
 		(fields_autoplaced yes)
-		(property "Reference" "C119"
+		(property "Reference" "C801"
 			(at 168.91 67.3099 0)
 			(effects
@@
 			(project "controller"
 				(path "/869bea87-c885-4ead-826b-3f34ceacafad/0e7b3f4d-646f-4949-ba8d-4e4489aa7d1d"
-					(reference "C119")
+					(reference "C801")
 					(unit 1)
 				)
@@
 		(on_board yes)
 		(dnp no)
-		(property "Reference" "TP126"
+		(property "Reference" "TP801"
 			(at 115.316 74.93 0)
 			(effects
@@
 			)
 		)
-		(property "Footprint" "TestPoint:TestPoint_Pad_1.0x1.0mm"
-			(at 123.19 82.55 0)
-			(effects
-				(font
-					(size 1.27 1.27)
-				)
-				(hide yes)
-			)
-		)
-		(property "Datasheet" "~"
-			(at 123.19 82.55 0)
-			(effects
-				(font
-					(size 1.27 1.27)
-				)
-				(hide yes)
-			)
-		)
-		(property "Description" "test point"
+		(property "Footprint" "5000"
+			(at 134.62 177.47 0)
+			(effects
+				(font
+					(size 1.27 1.27)
+				)
+				(justify left top)
+				(hide yes)
+			)
+		)
+		(property "Datasheet" "http://www.keyelco.com/product-pdf.cfm?p=1310"
+			(at 134.62 277.47 0)
+			(effects
+				(font
+					(size 1.27 1.27)
+				)
+				(justify left top)
+				(hide yes)
+			)
+		)
+		(property "Description" "KEYSTONE - 5001 - TEST POINT, CONNECTOR, BLACK"
 			(at 118.11 82.55 0)
 			(effects
@@
 					(size 1.27 1.27)
 				)
+				(hide yes)
+			)
+		)
+		(property "Height" ""
+			(at 134.62 477.47 0)
+			(effects
+				(font
+					(size 1.27 1.27)
+				)
+				(justify left top)
+				(hide yes)
+			)
+		)
+		(property "Manufacturer_Name" "Keystone Electronics"
+			(at 134.62 577.47 0)
+			(effects
+				(font
+					(size 1.27 1.27)
+				)
+				(justify left top)
+				(hide yes)
+			)
+		)
+		(property "Manufacturer_Part_Number" "5001"
+			(at 134.62 677.47 0)
+			(effects
+				(font
+					(size 1.27 1.27)
+				)
+				(justify left top)
+				(hide yes)
+			)
+		)
+		(property "Mouser Part Number" "534-5001"
+			(at 134.62 777.47 0)
+			(effects
+				(font
+					(size 1.27 1.27)
+				)
+				(justify left top)
+				(hide yes)
+			)
+		)
+		(property "Mouser Price/Stock" "https://www.mouser.co.uk/ProductDetail/Keystone-Electronics/5001?qs=q0tsjPZWdm%2FW0vdr%2FwowKg%3D%3D"
+			(at 134.62 877.47 0)
+			(effects
+				(font
+					(size 1.27 1.27)
+				)
+				(justify left top)
+				(hide yes)
+			)
+		)
+		(property "Arrow Part Number" "5001"
+			(at 134.62 977.47 0)
+			(effects
+				(font
+					(size 1.27 1.27)
+				)
+				(justify left top)
+				(hide yes)
+			)
+		)
+		(property "Arrow Price/Stock" "https://www.arrow.com/en/products/5001/keystone-electronics?utm_currency=USD&region=europe"
+			(at 134.62 1077.47 0)
+			(effects
+				(font
+					(size 1.27 1.27)
+				)
+				(justify left top)
 				(hide yes)
 			)
@@
 			(project "controller"
 				(path "/869bea87-c885-4ead-826b-3f34ceacafad/0e7b3f4d-646f-4949-ba8d-4e4489aa7d1d"
-					(reference "TP126")
+					(reference "TP801")
 					(unit 1)
 				)
@@
 		(dnp no)
 		(fields_autoplaced yes)
-		(property "Reference" "C122"
+		(property "Reference" "C804"
 			(at 180.34 115.5699 0)
 			(effects
@@
 			(project "controller"
 				(path "/869bea87-c885-4ead-826b-3f34ceacafad/0e7b3f4d-646f-4949-ba8d-4e4489aa7d1d"
-					(reference "C122")
+					(reference "C804")
 					(unit 1)
 				)
