File: hardware/controller/MEMORY.kicad_sch (KiCad schematic)
At the start: 8 parts, among them IC801 4677, IC802 W25Q256JVEIQ

Commit message: forgor
Parts:
- TP801, TP802: footprint 5000 -> SamacSys_Parts:5000
Other:
- note added: "Flash"
- note added: "Hierarchical Pins"
- note added: "PSRAM"
- note removed: "PSRAM and Flash"
- note removed: "these need decouping caps"
- moved on the sheet: C801, C802, C803, C804, IC801, IC802, TP801, TP802
