File: hardware/controller/USBC.kicad_sch (KiCad schematic)
At the start: 8 parts

Commit message: clean up DRC. need to add stitching vias and figure out why inner ground plane isnt connected to F.Cu pour
Parts:
- removed J102: ~, SamacSys_Parts:USB480003A, symbol Connector:USB_C_Receptacle_USB2.0_16P
- added J2: USB_C_Receptacle_USB2.0_16P, Connector_USB:USB_C_Receptacle_GCT_USB4105-xx-A_16P_TopMnt_Horizontal, symbol Connector:USB_C_Receptacle_USB2.0_16P
- renumbered D104 to D301, D105 to D302, D106 to D303, R104 to R301, R105 to R302, R106 to R303, R107 to R304
Connections:
- net CC1: now also J2.A5 (CC1)
- net CC2: now also J2.B5 (CC2)
- net D+: now also J2.A6 (D+), J2.B6 (D+)
- net D-: now also J2.A7 (D-), J2.B7 (D-)
- net GND: now also J2.A1 (GND), J2.A12 (GND), J2.B1 (GND), J2.B12 (GND), J2.S1 (SHIELD)
- net USBC_VBUS: now also J2.A4 (VBUS), J2.A9 (VBUS), J2.B4 (VBUS), J2.B9 (VBUS)
Other:
- note removed: "todo: check if need pull up resistor on data lines"
Changed lines of the file:
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@@
-		)
-	)
-	(text "todo: check if need pull up resistor on data lines"
-		(exclude_from_sim no)
-		(at 170.434 72.898 0)
-		(effects
-			(font
-				(size 10 10)
-			)
 		)
 	)
@@
 	)
 	(junction
-		(at 48.26 68.58)
+		(at 25.4 96.52)
 		(diameter 0)
 		(color 0 0 0 0)
 	)
 	(junction
-		(at 25.4 96.52)
+		(at 48.26 68.58)
 		(diameter 0)
 		(color 0 0 0 0)
@@
 		(dnp no)
 		(fields_autoplaced yes)
-		(property "Reference" "J102"
-			(at 33.02 46.99 0)
-			(effects
-				(font
-					(size 1.27 1.27)
-				)
-			)
-		)
-		(property "Value" "~"
-			(at 33.02 49.53 0)
-			(effects
-				(font
-					(size 1.27 1.27)
-				)
-			)
-		)
-		(property "Footprint" "SamacSys_Parts:USB480003A"
-			(at 59.69 163.5 0)
-			(effects
-				(font
-					(size 1.27 1.27)
-				)
-				(justify left top)
-				(hide yes)
-			)
-		)
-		(property "Datasheet" "https://gct.co/connector/usb4800"
-			(at 59.69 263.5 0)
-			(effects
-				(font
-					(size 1.27 1.27)
-				)
-				(justify left top)
-				(hide yes)
-			)
-		)
-		(property "Description" "USB Connectors USB2.0 Type C Rcpt, SMT, Hrz, 3.5mm elevated, 16 Pin"
+		(property "Reference" "J2"
+			(at 33.02 45.72 0)
+			(effects
+				(font
+					(size 1.27 1.27)
+				)
+			)
+		)
+		(property "Value" "USB_C_Receptacle_USB2.0_16P"
+			(at 33.02 48.26 0)
+			(effects
+				(font
+					(size 1.27 1.27)
+				)
+			)
+		)
+		(property "Footprint" "Connector_USB:USB_C_Receptacle_GCT_USB4105-xx-A_16P_TopMnt_Horizontal"
+			(at 36.83 68.58 0)
+			(effects
+				(font
+					(size 1.27 1.27)
+				)
+				(hide yes)
+			)
+		)
+		(property "Datasheet" "https://www.usb.org/sites/default/files/documents/usb_type-c.zip"
+			(at 36.83 68.58 0)
+			(effects
+				(font
+					(size 1.27 1.27)
+				)
+				(hide yes)
+			)
+		)
+		(property "Description" "USB 2.0-only 16P Type-C Receptacle connector"
 			(at 33.02 68.58 0)
 			(effects
@@
 			)
 		)
-		(property "Height" "5.58"
-			(at 59.69 463.5 0)
-			(effects
-				(font
-					(size 1.27 1.27)
-				)
-				(justify left top)
-				(hide yes)
-			)
-		)
-		(property "Mouser Part Number" "640-USB4800-03-A"
-			(at 59.69 563.5 0)
-			(effects
-				(font
-					(size 1.27 1.27)
-				)
-				(justify left top)
-				(hide yes)
-			)
-		)
-		(property "Mouser Price/Stock" "https://www.mouser.co.uk/ProductDetail/GCT/USB4800-03-A?qs=vvQtp7zwQdMkfG8vViEZoQ%3D%3D"
-			(at 59.69 663.5 0)
-			(effects
-				(font
-					(size 1.27 1.27)
-				)
-				(justify left top)
-				(hide yes)
-			)
-		)
-		(property "Manufacturer_Name" "GCT (GLOBAL CONNECTOR TECHNOLOGY)"
-			(at 59.69 763.5 0)
-			(effects
-				(font
-					(size 1.27 1.27)
-				)
-				(justify left top)
-				(hide yes)
-			)
-		)
-		(property "Manufacturer_Part_Number" "USB4800-03-A"
-			(at 59.69 863.5 0)
-			(effects
-				(font
-					(size 1.27 1.27)
-				)
-				(justify left top)
-				(hide yes)
-			)
+		(property "Mouser Stock/Price" "https://www.mouser.com/ProductDetail/Same-Sky/UJ20-C-H-G-SMT-1-P16-TR?qs=IKkN%2F947nfA6nby92vSKkw%3D%3D&srsltid=AfmBOoqgW8J1ZzVCat00JQQ9Um36NnE84vN6B7UjXbLiSONBgxyj8db_"
+			(at 33.02 68.58 0)
+			(effects
+				(font
+					(size 1.27 1.27)
+				)
+				(hide yes)
+			)
+		)
+		(pin "B4"
+		)
+		(pin "A5"
+		)
+		(pin "A8"
+		)
+		(pin "A9"
+		)
+		(pin "B5"
+		)
+		(pin "B6"
+		)
+		(pin "A6"
+		)
+		(pin "B12"
+		)
+		(pin "S1"
+		)
+		(pin "A12"
+		)
+		(pin "B1"
+		)
+		(pin "A7"
+		)
+		(pin "B8"
+		)
+		(pin "A4"
 		)
 		(pin "A1"
 		)
-		(pin "A9"
-		)
-		(pin "A4"
-		)
-		(pin "S1"
+		(pin "B9"
 		)
 		(pin "B7"
-		)
-		(pin "B5"
-		)
-		(pin "A7"
-		)
-		(pin "B12"
-		)
-		(pin "B1"
-		)
-		(pin "A12"
-		)
-		(pin "A6"
-		)
-		(pin "B8"
-		)
-		(pin "A5"
-		)
-		(pin "A8"
-		)
-		(pin "B9"
-		)
-		(pin "B6"
-		)
-		(pin "B4"
 		)
 		(instances
 			(project ""
 				(path "/869bea87-c885-4ead-826b-3f34ceacafad/26d17bc2-e2ae-44e6-8fc3-d458d6e51b4a"
-					(reference "J102")
+					(reference "J2")
 					(unit 1)
 				)
@@
 		(dnp no)
 		(fields_autoplaced yes)
-		(property "Reference" "#PWR0121"
+		(property "Reference" "#PWR0301"
 			(at 25.4 104.14 0)
 			(effects
@@
 			(project ""
 				(path "/869bea87-c885-4ead-826b-3f34ceacafad/26d17bc2-e2ae-44e6-8fc3-d458d6e51b4a"
-					(reference "#PWR0121")
+					(reference "#PWR0301")
 					(unit 1)
 				)
@@
 		(dnp no)
 		(fields_autoplaced yes)
-		(property "Reference" "#PWR0123"
+		(property "Reference" "#PWR0303"
 			(at 73.66 66.04 0)
 			(effects
@@
 			(project ""
 				(path "/869bea87-c885-4ead-826b-3f34ceacafad/26d17bc2-e2ae-44e6-8fc3-d458d6e51b4a"
-					(reference "#PWR0123")
+					(reference "#PWR0303")
 					(unit 1)
 				)
@@
 		(dnp no)
 		(fields_autoplaced yes)
-		(property "Reference" "D105"
+		(property "Reference" "D302"
 			(at 93.98 76.1999 90)
 			(effects
@@
 			(project "controller"
 				(path "/869bea87-c885-4ead-826b-3f34ceacafad/26d17bc2-e2ae-44e6-8fc3-d458d6e51b4a"
-					(reference "D105")
+					(reference "D302")
 					(unit 1)
 				)
@@
 		(on_board yes)
 		(dnp no)
-		(property "Reference" "R104"
+		(property "Reference" "R301"
 			(at 57.404 56.388 90)
 			(effects
@@
 			(project ""
 				(path "/869bea87-c885-4ead-826b-3f34ceacafad/26d17bc2-e2ae-44e6-8fc3-d458d6e51b4a"
-					(reference "R104")
+					(reference "R301")
 					(unit 1)
 				)
@@
 		(dnp no)
 		(fields_autoplaced yes)
-		(property "Reference" "D106"
+		(property "Reference" "D303"
 			(at 128.27 59.6899 90)
 			(effects
@@
 			(project "controller"
 				(path "/869bea87-c885-4ead-826b-3f34ceacafad/26d17bc2-e2ae-44e6-8fc3-d458d6e51b4a"
-					(reference "D106")
+					(reference "D303")
 					(unit 1)
 				)
@@
 		(dnp no)
 		(fields_autoplaced yes)
-		(property "Reference" "#PWR0124"
+		(property "Reference" "#PWR0304"
 			(at 91.44 87.63 0)
 			(effects
@@
 			(project "controller"
 				(path "/869bea87-c885-4ead-826b-3f34ceacafad/26d17bc2-e2ae-44e6-8fc3-d458d6e51b4a"
-					(reference "#PWR0124")
+					(reference "#PWR0304")
 					(unit 1)
 				)
@@
 		(dnp no)
 		(fields_autoplaced yes)
-		(property "Reference" "#PWR0125"
+		(property "Reference" "#PWR0305"
 			(at 125.73 87.63 0)
 			(effects
@@
 			(project ""
 				(path "/869bea87-c885-4ead-826b-3f34ceacafad/26d17bc2-e2ae-44e6-8fc3-d458d6e51b4a"
-					(reference "#PWR0125")
+					(reference "#PWR0305")
 					(unit 1)
 				)
@@
 		(on_board yes)
 		(dnp no)
-		(property "Reference" "R107"
+		(property "Reference" "R304"
 			(at 107.95 73.406 90)
 			(effects
@@
 			(project "controller"
 				(path "/869bea87-c885-4ead-826b-3f34ceacafad/26d17bc2-e2ae-44e6-8fc3-d458d6e51b4a"
-					(reference "R107")
+					(reference "R304")
 					(unit 1)
 				)
@@
 		(dnp no)
 		(fields_autoplaced yes)
-		(property "Reference" "D104"
+		(property "Reference" "D301"
 			(at 59.69 76.1999 90)
 			(effects
@@
 			(project "controller"
 				(path "/869bea87-c885-4ead-826b-3f34ceacafad/26d17bc2-e2ae-44e6-8fc3-d458d6e51b4a"
-					(reference "D104")
+					(reference "D301")
 					(unit 1)
 				)
@@
 		(on_board yes)
 		(dnp no)
-		(property "Reference" "R106"
+		(property "Reference" "R303"
 			(at 107.95 66.548 90)
 			(effects
@@
 			(project ""
 				(path "/869bea87-c885-4ead-826b-3f34ceacafad/26d17bc2-e2ae-44e6-8fc3-d458d6e51b4a"
-					(reference "R106")
+					(reference "R303")
 					(unit 1)
 				)
@@
 		(on_board yes)
 		(dnp no)
-		(property "Reference" "R105"
+		(property "Reference" "R302"
 			(at 67.31 58.928 90)
 			(effects
@@
 			(project "controller"
 				(path "/869bea87-c885-4ead-826b-3f34ceacafad/26d17bc2-e2ae-44e6-8fc3-d458d6e51b4a"
-					(reference "R105")
+					(reference "R302")
 					(unit 1)
 				)
@@
 		(dnp no)
 		(fields_autoplaced yes)
-		(property "Reference" "#PWR0122"
+		(property "Reference" "#PWR0302"
 			(at 57.15 87.63 0)
 			(effects
@@
 			(project "controller"
 				(path "/869bea87-c885-4ead-826b-3f34ceacafad/26d17bc2-e2ae-44e6-8fc3-d458d6e51b4a"
-					(reference "#PWR0122")
+					(reference "#PWR0302")
 					(unit 1)
 				)

Commit message: save before axing motor driver ic's
Parts:
- J2: Mouser Stock/Price https://www.mouser.com/ProductDetail/Same-Sky/UJ20-C-H-G-SM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 -> https://www.mouser.co.uk/ProductDetail/Same-Sky/UJ20-C-H-G-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
- R303, R304: Mouser Price/Stock https://www.mouser.com/Search/Refine.aspx?Keyword=71-CRCW04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 -> https://www.mouser.co.uk/Search/Refine.aspx?Keyword=71-CRCW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
Changed lines of the file:
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@@
 			)
 		)
-		(property "Mouser Stock/Price" "https://www.mouser.com/ProductDetail/Same-Sky/UJ20-C-H-G-SMT-1-P16-TR?qs=IKkN%2F947nfA6nby92vSKkw%3D%3D&srsltid=AfmBOoqgW8J1ZzVCat00JQQ9Um36NnE84vN6B7UjXbLiSONBgxyj8db_"
+		(property "Mouser Stock/Price" "https://www.mouser.co.uk/ProductDetail/Same-Sky/UJ20-C-H-G-SMT-1-P16-TR?qs=IKkN%2F947nfA6nby92vSKkw%3D%3D&srsltid=AfmBOoqgW8J1ZzVCat00JQQ9Um36NnE84vN6B7UjXbLiSONBgxyj8db_"
 			(at 33.02 68.58 0)
 			(effects
@@
 			)
 		)
-		(property "Mouser Price/Stock" "https://www.mouser.com/Search/Refine.aspx?Keyword=71-CRCW0402J-27"
+		(property "Mouser Price/Stock" "https://www.mouser.co.uk/Search/Refine.aspx?Keyword=71-CRCW0402J-27"
 			(at 704.14 57.15 0)
 			(effects
@@
 			)
 		)
-		(property "Mouser Price/Stock" "https://www.mouser.com/Search/Refine.aspx?Keyword=71-CRCW0402J-27"
+		(property "Mouser Price/Stock" "https://www.mouser.co.uk/Search/Refine.aspx?Keyword=71-CRCW0402J-27"
 			(at 704.14 54.61 0)
 			(effects
