File: hardware/drone/USB_UART.kicad_sch (KiCad schematic)
At the start: 7 parts, among them IC102 CP2102N-A02-GQFN28

Commit message: save before axing motor driver ic's
Parts:
- R118: Mouser Price/Stock https://www.mouser.com/ProductDetail/Vishay/CRCW060322K1FKE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 -> https://www.mouser.co.uk/ProductDetail/Vishay/CRCW060322K1F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
Changed lines of the file:
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@@
 			)
 		)
-		(property "Mouser Price/Stock" "https://www.mouser.com/ProductDetail/Vishay/CRCW060322K1FKEBC?qs=wd5RIQLrsJgpX5GYef5UHQ%3D%3D"
+		(property "Mouser Price/Stock" "https://www.mouser.co.uk/ProductDetail/Vishay/CRCW060322K1FKEBC?qs=wd5RIQLrsJgpX5GYef5UHQ%3D%3D"
 			(at 92.71 121.92 90)
 			(effects
